File: presentation/meetings/2026-10-21-v2/interposer/project/XEM_Interposer_V23_PCM_Switch.kicad_pcb (KiCad board)
At the start: 6 copper layers, 83 x 53 mm, 57 parts, among them J1 PKS019-4011-0, SW1 JS102011SABN, U1 TPS26600PWPR, U2 TPS62162DSGR, U3 TPS259470ARPWR, U5 TMUX1574PWR, U6 TLV6700DDCR, U7 SN74LVC1G97DBVR

Commit message: Refresh meeting interposer to V23 and improve carrier views
Parts:
- C20, C21, C22: value 100 nF / 10 V -> 100 nF / 16 V
- C5, C7: value 1 µF / 10 V -> 1 µF / 25 V
- C6: value 3.3 nF / 10 V -> 3.3 nF / 50 V
- SW1: value JS102011SABN -> PCM12SMTBR; footprint SwitchAccess:SW_SPDT_CK_JS102011SABN -> SwitchAccess:SW_SPDT_CK_PCM12SMTBR
- moved SW1 0.55 mm to (180.7, 115.0)
Connections:
- SW1 pad 1: GND -> unconnected-(SW1-Pad1)
Routing:
- net GND: track 193.3 -> 191.6 mm
- net /JTAG_REMOTE_SELECT: track 88.0 -> 89.1 mm
Other:
- board text added: "V23 WIDER POWER / PARALLEL ACCESS | 2.4mm stack provisional"
- board text added: "XEM INTERPOSER V23"
- board text removed: "V20 WIDER POWER / PARALLEL ACCESS | 2.4mm stack provisional"
- board text removed: "XEM INTERPOSER V20"
